File: Naz80-b/Naz80-b/Naz80-b.kicad_pcb (KiCad board)
At the start: 2 copper layers, 68 parts, among them J1 Display Connector, Q1 2N3906, Q2 2N3906, Q3 2N3906, Q4 2N3906, Q5 2N3906, Q6 2N3906, Q7 2N3906, Q8 2N3906, Q9 2N3906, SW1 SW_Push, U1 74LS14, U10 W27C512, U11 HM62256BLP, U12 74LS04, U2 74LS04, U3 74LS32, U4 Z80CPU, U5 74LS139, U6 82C55A, U7 W27C512, U8 MC68B50, U9 HM62256BLP, X1 CXO_DIP8

Commit message: Changed UART to Z84 SIO-2 and added Z8O PIO
Parts:
- removed J1: Display Connector, Connector_PinHeader_2.54mm:PinHeader_1x16_P2.54mm_Horizontal
- removed R22: 330, Resistor_THT:R_Axial_DIN0411_L9.9mm_D3.6mm_P12.70mm_Horizontal
- removed U10: W27C512, Socket:DIP_Socket-28_W11.9_W12.7_W15.24_W17.78_W18.5_3M_228-1277-00-0602J
- removed U11: HM62256BLP, Package_DIP:DIP-28_W15.24mm
- removed U12: 74LS04, Package_DIP:DIP-16_W7.62mm_LongPads
- moved U4 135.4 mm to (30.5, 61.0)
- moved U7 126.7 mm to (58.4, 17.8)
- moved U9 124.1 mm to (30.5, 17.8)
- moved U2 74.5 mm to (104.1, 61.0)
- moved U6 69.6 mm to (73.7, 109.2)
- moved U8 58.3 mm to (85.5, 22.9)
- moved U1 53.6 mm to (121.9, 94.9)
- moved U5 20.2 mm to (133.5, 94.9)
- moved U3 13.6 mm to (87.0, 61.0)
Connections:
- net /~{M_R} renamed /~{M_OE}
- U2 pad 2: Net-(U7-*CE) -> Net-(U9-~{CS})
- U2 pad 3: unconnected-(U2-Pad3) -> ~{IORQ}
- U2 pad 4: unconnected-(U2-Pad4) -> Net-(U8-E)
- U3 pad 11: /~{IO_W} -> /~{IO_WE}
- U3 pad 12: /~{WR} -> ~{IORQ}
- U3 pad 13: ~{IORQ} -> /~{WR}
- U3 pad 4: /~{WR} -> /~{MREQ}
- U3 pad 5: /~{MREQ} -> /~{WR}
- U3 pad 6: /~{M_W} -> /~{M_WE}
- U3 pad 8: /~{IO_R} -> /~{IO_OE}
- U5 pad 1: ~{IORQ} -> (no net)
- U5 pad 10: unconnected-(U5B-O2-Pad10) -> (no net)
- U5 pad 11: unconnected-(U5B-O1-Pad11) -> (no net)
- U5 pad 12: unconnected-(U5B-O0-Pad12) -> (no net)
- U5 pad 13: /A5 -> (no net)
- U5 pad 14: /A4 -> (no net)
- U5 pad 15: ~{IORQ} -> (no net)
- U5 pad 2: /A6 -> (no net)
- U5 pad 3: /A7 -> (no net)
- U5 pad 4: /PIO_CE -> (no net)
- U5 pad 5: /UART_CS -> (no net)
- U5 pad 6: unconnected-(U5A-O2-Pad6) -> (no net)
- U5 pad 7: unconnected-(U5A-O3-Pad7) -> (no net)
- U5 pad 9: unconnected-(U5B-O3-Pad9) -> (no net)
- U6 pad 1: /D3 -> (no net)
- U6 pad 10: unconnected-(U6-PC7-Pad10) -> (no net)
- U6 pad 11: unconnected-(U6-PC6-Pad11) -> (no net)
- U6 pad 12: unconnected-(U6-PC5-Pad12) -> (no net)
- U6 pad 13: unconnected-(U6-PC4-Pad13) -> (no net)
- U6 pad 14: unconnected-(U6-PC0-Pad14) -> (no net)
- U6 pad 15: unconnected-(U6-PC1-Pad15) -> (no net)
- U6 pad 16: unconnected-(U6-PC2-Pad16) -> (no net)
- U6 pad 17: unconnected-(U6-PC3-Pad17) -> (no net)
- U6 pad 18: unconnected-(U6-PB0-Pad18) -> (no net)
- U6 pad 19: unconnected-(U6-PB1-Pad19) -> (no net)
- U6 pad 2: /D2 -> (no net)
- U6 pad 20: unconnected-(U6-PB2-Pad20) -> (no net)
- U6 pad 21: unconnected-(U6-PB3-Pad21) -> (no net)
- U6 pad 22: unconnected-(U6-PB4-Pad22) -> (no net)
- U6 pad 23: unconnected-(U6-PB5-Pad23) -> (no net)
- U6 pad 24: unconnected-(U6-PB6-Pad24) -> (no net)
- U6 pad 25: unconnected-(U6-PB7-Pad25) -> (no net)
- U6 pad 26: +5V -> (no net)
- U6 pad 27: /D7 -> (no net)
- U6 pad 28: /D6 -> (no net)
- U6 pad 29: /D5 -> (no net)
- U6 pad 3: /D1 -> (no net)
- U6 pad 30: /D4 -> (no net)
- U6 pad 31: /D3 -> (no net)
- U6 pad 32: /D2 -> (no net)
- U6 pad 33: /D1 -> (no net)
- U6 pad 34: /D0 -> (no net)
- U6 pad 35: /RESET -> (no net)
- U6 pad 36: /~{IO_W} -> (no net)
- U6 pad 37: unconnected-(U6-PA7-Pad37) -> (no net)
- U6 pad 38: /E -> (no net)
- U6 pad 39: /RW -> (no net)
- U6 pad 4: /D0 -> (no net)
- U6 pad 40: /RS -> (no net)
- U6 pad 5: /~{IO_R} -> (no net)
- U6 pad 6: /PIO_CE -> (no net)
- U6 pad 7: GND -> (no net)
- U6 pad 8: /A1 -> (no net)
- U6 pad 9: /A0 -> (no net)
- U7 pad 20: Net-(U7-*CE) -> /A15
- U8 pad 13: /~{IO_W} -> /~{IO_WE}
- U8 pad 14: ~{IORQ} -> Net-(U8-E)
- U9 pad 20: /A15 -> Net-(U9-~{CS})
Routing:
- net /A6: track 129.8 -> 0.00 mm
- net /A7: track 106.7 -> 0.00 mm
- net /~{M_OE}: track 91.4 -> 0.00 mm
- net /A1: track 90.4 -> 0.00 mm
- net /D6: track 90.0 -> 0.00 mm
- net /D5: track 84.1 -> 0.00 mm
- net GND: track 82.0 -> 0.00 mm
- net /D4: track 78.4 -> 0.00 mm
- net /D2: track 77.2 -> 0.00 mm
- net /D1: track 77.2 -> 0.00 mm
- net /D0: track 77.2 -> 0.00 mm
- net /~{IO_R}: track 70.3 -> 0.00 mm
- net /~{M_W}: track 61.6 -> 0.00 mm
- net /A13: track 51.3 -> 0.00 mm
- net /A4: track 51.0 -> 0.00 mm
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