File: Naz80-b/Naz80-b/Naz80-b.kicad_sch (KiCad schematic)
At the start: 27 parts, among them J1 Conn_01x16, SW1 SW_Push, U1 74LS14, U10 74LS138, U2 74LS04, U3 74LS32, U4 Z80CPU, U5 74LS139, U6 82C55A, U7 W27C512, U8 MC68B50, U9 HM62256BLP, X1 CXO_DIP8

Commit message: Changed UART to Z84 SIO-2 and added Z8O PIO
Parts:
- removed U8: MC68B50, Package_DIP:DIP-24_W15.24mm, symbol Interface_UART:MC68B50
- added C11, C12: 0.1uF, Capacitor_THT:C_Radial_D6.3mm_H7.0mm_P2.50mm, symbol Device:C
- added U11: Z80SIO2, Package_DIP:DIP-40_W15.24mm, symbol Naz80:Z80SIO2
- added U12: (no value), Package_DIP:DIP-40_W15.24mm, symbol Naz80:DS12885
- added U8: Z8420, Package_DIP:DIP-40_W15.24mm, symbol Interface:Z8420
- JP1: now in the parts list
- U4: symbol CPU:Z80CPU -> Naz80:Z80CPU
Connections:
- net ~{M_W} is gone; now on net ~{M_WE}: U9.27 (~{WE})
- net +5V: now also U10.16 (VCC), C11.1, C12.1, U11.9 (+5V), U8.26 (VCC); no longer U4.24 (~{WAIT}), U4.25 (~{BUSRQ})
- net A0: now also J1.9 (Pin_9), U11.34 (B/~{A}), U8.6 (B/~{A}); no longer J1.11 (Pin_11)
- net A1: now also U11.33 (C/~{D}), U8.5 (C/~{D})
- net A5: no longer U10.3 (A2)
- net A7: now also U10.3 (A2)
- net CLK: now also U11.20 (CLK), U8.25 (CLK)
- net D0: now also U11.40 (D0), U8.19 (D0)
- net D1: now also U11.1 (D1), U8.20 (D1)
- net D2: now also U11.39 (D2), U8.1 (D2)
- net D3: now also U11.2 (D3), U8.40 (D3)
- net D4: now also U11.38 (D4), U8.39 (D4)
- net D5: now also U11.3 (D5), U8.38 (D5)
- net D6: now also U11.37 (D6), U8.3 (D6)
- net D7: now also U11.4 (D7), U8.2 (D7)
- net GND: now also U10.8 (GND), C11.2, C12.2, U11.31 (GND), U8.11 (GND)
- net RESET: no longer U6.35 (RESET)
- net ~{INT}: now also U11.5 (~{INT})
- net ~{IORQ}: now also U11.36 (~{IORQ}), U8.23 (~{INT}), U8.36 (~{IORQ})
- net ~{IO_DISP}: no longer J1.9 (Pin_9)
- net ~{M1}: now also U11.8 (~{M1}), U8.37 (~{M1})
- net ~{M_OE}: no longer U3.3
- net ~{M_WE}: no longer U3.6
- net ~{RD}: now also U11.32 (~{RD}), U8.35 (~{RD})
- net ~{RESET}: now also U2.5, U11.21 (~{RESET})
- net ~{PRIN_EN}: now reaches U10.12 (O3)
- net ~{PRIN_EN}: now also U8.4 (~{CE})
- net ~{BUSACK}: now reaches U4.23 (~{BUSACK})
- net at U2.6: now also U6.35 (RESET)
- net PIO_CE renamed ~{IO_PIO}
- net UART_CS renamed ~{IO_UART}
- net ~{IO_OE} renamed ~{IO_RD}
- net ~{IO_WE} renamed ~{IO_WR}
- new net: U11.7 (IEO), U8.24 (IEI)
- new net ~{BUSRQ}: U4.25 (~{BUSRQ})
- new net ~{MEM_WR}: U3.6
- new net ~{M_RD}: U3.3
- new net ~{PRN_EN}: J1.11 (Pin_11)
- new net ~{UART_EN}: U11.35 (~{CE})
- new net ~{WAIT}: U4.24 (~{WAIT})
- no-connect marks 37 -> 29
Other:
- note added: "32k Ram"
- note added: "64K Rom with 32K split"
- moved on the sheet: C10, C6, C7, C8, C9, J1, U10, U1C, U1D, U1E, U1F, U2B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

Commit message: Redesign of board
Parts:
- removed C5: 0.1uF, Capacitor_THT:C_Radial_D6.3mm_H7.0mm_P2.50mm, symbol Device:C
- removed JP1: ROM BANK Selector, Connector_PinHeader_2.54mm:PinHeader_1x03_P2.54mm_Horizontal, symbol Jumper:Jumper_3_Open
- removed U12: (no value), Package_DIP:DIP-40_W15.24mm, symbol Naz80:DS12885
- removed U2: 74LS04, Package_DIP:DIP-16_W7.62mm_LongPads, symbol 74xx:74LS04
- removed U3: 74LS32, Package_DIP:DIP-16_W7.62mm_LongPads, symbol 74xx:74LS32
- removed U6: 82C55A, Package_DIP:DIP-40_W15.24mm, symbol Interface:82C55A
- removed X1: CXO_DIP8, Oscillator:Oscillator_DIP-8, symbol Oscillator:CXO_DIP8
- added D2: LED, LED_THT:LED_D5.0mm, symbol Device:LED
- added J3, J4: Conn_01x07, symbol Connector_Generic:Conn_01x07
- added J5: Conn_01x03, symbol Connector_Generic:Conn_01x03
- added J6, J7: Conn_01x07, symbol Connector_Generic:Conn_01x10
- added R11, R4, R5, R6: 4.7k, symbol Device:R
- added R3: 330, Resistor_THT:R_Axial_DIN0411_L9.9mm_D3.6mm_P12.70mm_Horizontal, symbol Device:R
- added U3: 74HC04, symbol 74xx:74HC04
- added U6: 74HC00, Module:Arduino_Nano, symbol 74xx:74HC00
- added Y3: ACO-8.0 MHz, Oscillator:Oscillator_DIP-14, symbol Oscillator:ACO-xxxMHz
- added Y4: ACO-7.3728MHz, Oscillator:Oscillator_DIP-14, symbol Oscillator:ACO-xxxMHz
Connections:
- net ~{IO_PIO} is gone; now on net ~{IO_UART}: U10.15 (O0)
- net ~{M_OE} is gone; now on net ~{RD}: U7.22 (*OE/VPP), U9.22 (~{OE})
- net ~{PRN_EN} is gone; now on net ~{IO_DISP}: J1.11 (Pin_11)
- net +5V: now also U10.6 (E3), U11.6 (IEI), J5.1 (Pin_1), R11.2, R3.2, R4.1, R5.1, R6.1, U3.14 (VCC), Y3.14 (Vcc), Y4.14 (Vcc)
- net A15: now also U3.13, U6.1; no longer U7.20 (*CE)
- net CLK: now also Y3.8 (OUT)
- net GND: now also U1.11, U1.13, U1.5, U1.9, U10.4 (E1), D2.1 (K), J3.7 (Pin_7), J4.7 (Pin_7), J5.3 (Pin_3), U3.7 (GND), Y3.7 (GND), Y4.7 (GND)
- net ~{BUSRQ}: now also R6.2
- net ~{IORQ}: no longer U10.4 (E1), U10.5 (E2)
- net ~{IO_DISP}: now also U10.14 (O1); no longer U10.13 (O2)
- net ~{IO_UART}: no longer U10.14 (O1)
- net ~{M1}: no longer U10.6 (E3)
- net ~{MREQ}: now also U3.11
- net ~{NMI}: now also R4.2
- net ~{PRIN_EN}: now also U10.13 (O2); no longer U10.12 (O3)
- net ~{WAIT}: now also R5.2
- net ~{WR}: now also J1.10 (Pin_10)
- net at U8.10 (PA4): now also J6.5 (Pin_5)
- net at U8.12 (PA3): now also J6.4 (Pin_4)
- net at U8.13 (PA2): now also J6.3 (Pin_3)
- net at U8.14 (PA1): now also J6.2 (Pin_2)
- net at U8.15 (PA0): now also J6.1 (Pin_1)
- net at U8.16 (~{ASTB}): now also J6.10 (Pin_10)
- net at U8.17 (~{BSTB}): now also J7.10 (Pin_10)
- net at U8.18 (ARDY): now also J6.9 (Pin_9)
- net at U8.21 (BRDY): now also J7.9 (Pin_9)
- net at U8.27 (PB0): now also J7.1 (Pin_1)
- net at U8.28 (PB1): now also J7.2 (Pin_2)
- net at U8.29 (PB2): now also J7.3 (Pin_3)
- net at U8.30 (PB3): now also J7.4 (Pin_4)
- net at U8.31 (PB4): now also J7.5 (Pin_5)
- net at U8.32 (PB5): now also J7.6 (Pin_6)
- net at U8.33 (PB6): now also J7.7 (Pin_7)
- net at U8.34 (PB7): now also J7.8 (Pin_8)
- net at U8.7 (PA7): now also J6.8 (Pin_8)
- net at U8.8 (PA6): now also J6.7 (Pin_7)
- net at U8.9 (PA5): now also J6.6 (Pin_6)
- net ~{RAM_CS}: now reaches U9.20 (~{CS})
- net ~{RAM_CS}: now also U6.3
- net at U11.11 (~{SYNCA}): now also R11.1
- net RxDA: now reaches U11.12 (RxDA)
- net RxDA: now also J3.1 (Pin_1)
- net CLK_SIO: now reaches U11.13 (~{RxCA})
- net CLK_SIO: now also U11.14 (~{TxCA}), U11.27 (~{TxCB}), U11.28 (~{RxCB}), Y4.8 (OUT)
- net TxDA: now reaches U11.15 (TxDA)
- net TxDA: now also J3.2 (Pin_2)
- net ~{DTRA}: now reaches U11.16 (~{DTRA})
- net ~{DTRA}: now also J3.5 (Pin_5)
- net ~{RTSA}: now reaches U11.17 (~{RTSA})
- net ~{RTSA}: now also J3.3 (Pin_3)
- net ~{CTSA}: now reaches U11.18 (~{CTSA})
- net ~{CTSA}: now also J3.4 (Pin_4)
- net ~{DCDA}: now reaches U11.19 (~{DCDA})
- net ~{DCDA}: now also J3.6 (Pin_6)
- net ~{DCDB}: now reaches U11.22 (~{DCDB})
- net ~{DCDB}: now also J4.6 (Pin_6)
- net ~{CTSB}: now reaches U11.23 (~{CTSB})
- net ~{RTSB}: now reaches U11.24 (~{RTSB})
- net ~{DTRB}: now reaches U11.25 (~{DTRB})
- net TxDB: now reaches U11.26 (TxDB)
- net TxDB: now also J4.2 (Pin_2)
- net RxDB: now reaches U11.29 (RxDB)
- net RxDB: now also J4.1 (Pin_1)
- net RB: no longer names the net of U7.1 (A15)
- net RB: now also J5.2 (Pin_2)
- net ~{M_WE} renamed ~{RW}
- net ~{RW}: no longer J1.10 (Pin_10)
- new net: U3.10, U6.2, U6.4
- new net: U3.12, U6.5
- new net: D2.2 (A), R3.1
- new net ~{IO_RQ}: U10.5 (E2)
- new net ~{ROM_CS}: U6.6, U7.20 (*CE)
- no-connect marks 29 -> 14
Other:
- removed sheet Indicators
- note added: "0x8000 - 0xFFFF"
- note added: "64K Rom with 32K split 0x0000 - 0xCFFF 0xD000 - 0xFFFF"
- note added: "Basic Memory Decode"
- note added: "CPU"
- note added: "Display"
- note added: "High ROM"
- note added: "IO Decode"
- note added: "IO Devices"
- note added: "Lcd Module - Datasheet"
- note added: "Low ROM"
- note added: "Memory"
- note added: "Oscillators"
- note added: "Printer Port"
- note added: "Reset Circuit"
- note added: "Serial Port"
- note added: "UART"
- note removed: "64K Rom with 32K split"
- note removed: "IO Request"
- note removed: "Memory Request"
- note removed: "https://cdn.soselectronic.com/productdata/03/fd/c9895a2a/dem-16215-syh-ly.pdf"
- company: (none) -> A Thousand Projects
- title: (none) -> Naz80B
- moved on the sheet: C10, C11, C12, C6, C7, C8, C9, J1, U10, U11, U1C, U1D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
