File: Naz80-b/Naz80-b.kicad_sch (KiCad schematic)
At the start: 39 parts, among them J1 Conn_01x16, J3 Conn_01x07, J4 Conn_01x07, J5 Conn_01x03, J6 Conn_01x07, J7 Conn_01x07, SW1 SW_Push, U1 74LS14, U10 74LS138, U11 Z80SIO2, U3 74HC04, U4 Z80CPU, U5 74LS139, U6 74HC00, U7 W27C512, U8 Z8420, U9 HM62256BLP, Y3 ACO-8.0 MHz, Y4 ACO-7.3728MHz

Commit message: Corrected Memory mappings
Other:
- note added: "32k Ram 0x8000 - 0xFFFF"
- note added: "64K Rom with 32K split 0x0000 - 0x7FFF 0x8000 - 0xFFFF 0x0000 - 7FFFF (addressable)"
- note added: "POI : 0x20 - 0xE0"
- note removed: "0x8000 - 0xFFFF"
- note removed: "32k Ram"
- note removed: "64K Rom with 32K split 0x0000 - 0xCFFF 0xD000 - 0xFFFF"
- note removed: "POI : 0x80 - 0x83"
Changed lines of the file:
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@@
 		)
 	)
-	(text "0x8000 - 0xFFFF"
+	(text ""
 		(exclude_from_sim no)
 		(at 377.19 94.488 0)
@@
 		)
 	)
-	(text "64K Rom with 32K split\n\n0x0000 - 0xCFFF\n0xD000 - 0xFFFF"
+	(text "64K Rom with 32K split\n\n0x0000 - 0x7FFF\n0x8000 - 0xFFFF\n\n0x0000 - 7FFFF (addressable)"
 		(exclude_from_sim no)
-		(at 318.516 94.742 0)
+		(at 316.23 93.726 0)
 		(effects
 			(font
@@
 				(bold yes)
 			)
+			(justify left)
 		)
 	)
@@
 		)
 	)
-	(text "32k Ram"
+	(text "32k Ram\n\n0x8000 - 0xFFFF"
 		(exclude_from_sim no)
-		(at 377.952 91.44 0)
+		(at 367.03 92.456 0)
 		(effects
 			(font
@@
 				(bold yes)
 			)
+			(justify left)
 		)
 	)
-	(text "POI : 0x80 - 0x83"
+	(text "POI : 0x20 - 0xE0"
 		(exclude_from_sim no)
 		(at 211.074 193.802 0)
